File: idp/idp-valid.kicad_pcb (KiCad board)
At the start: 2 copper layers, 302.3 x 247 mm, 307 parts, among them J1 PinHeader_2x17_P2.54mm_Vertic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, J2 PinHeader_2x32_P2.54mm_Vertic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, J3 PinHeader_1x03_P2.54mm_Vertic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, J4 PinHeader_2x25_P2.54mm_Vertic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, J5 PinHeader_1x05_P2.54mm_Vertic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, J6 PinHeader_2x20_P2.54mm_Vertic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, J7 PinHeader_2x13_P2.54mm_Vertic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, J8 PinHeader_2x13_P2.54mm_Vertic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, J9 PinHeader_2x13_P2.54mm_Vertic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, X10 Partner_Molex_Mega-Fit_76829-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, Y1 8.000, Y2 32.768 kHZ, Y3 1.8432

Commit message: Adjusts track and via sizes
Routing:
- net (no net): vias 1042 -> 1039
