File: pcb/idp.kicad_pcb (KiCad board)
At the start: 2 copper layers, 302.3 x 247 mm, 308 parts, among them Y1 8MHz, Y2 32.768kHz, Y3 1.8432MHz

Commit message: Assigns refs CX1-CX41 to decoupling caps
Parts:
- renumbered CX to CX1, CX to CX10, CX to CX11, CX to CX12, CX to CX13, CX to CX14, CX to CX15, CX to CX16, CX to CX17, CX to CX18, CX to CX19, CX to CX2, CX to CX20, CX to CX21, CX to CX22, CX to CX23, CX to CX24, CX to CX25, CX to CX26, CX to CX27, CX to CX28, CX to CX29, CX to CX3, CX to CX30, CX to CX31, CX to CX32, CX to CX33, CX to CX34, CX to CX35, CX to CX36, CX to CX37, CX to CX38, CX to CX39, CX to CX4, CX to CX40, CX to CX41, CX to CX5, CX to CX6, CX to CX7, CX to CX8, CX to CX9
