File: pcb/idp.kicad_pcb (KiCad board)
At the start: 2 copper layers, 302.3 x 247 mm, 308 parts, among them Y1 8MHz, Y2 32.768kHz, Y3 1.8432MHz

Commit message: Assigns nets to remaining pads
Parts:
- BAT: value 3.6V -> (none)
- C1, C2, C3, C4: value 100μ -> (none)
- C102, C7: value 2.2n -> (none)
- C103, C110: value 391 -> (none)
- C17: value 68p -> (none)
- C18: value 82p -> (none)
- C20, C8: value 68μ -> (none)
- C21, C22: value 20p -> (none)
- C300: value 331 -> (none)
- C301: value 680n -> (none)
- C5, C6: value 1n -> (none)
- CX1, CX10, CX11, CX12, CX13, CX14, CX15, CX16, CX17, CX18, CX19, CX2, CX20, CX21, CX22, CX23, CX24, CX25, CX26, CX27, CX28, CX29, CX3, CX30, CX31, CX32, CX33, CX34, CX35, CX36, CX37, CX38, CX39, CX4, CX40, CX41, CX5, CX6, CX7, CX8, CX9: value 104 -> (none)
- E1, E58: value LS123 -> (none)
- E10, E79, E92, E93: value LS30 -> (none)
- E100, E101, E59, E60, E61, E62, E71, E72, E73, E74, E85, E86, E87, E88, E98, E99: value M3764A-15 -> (none)
- E102: value LS86 -> (none)
- E103, E104, E106, E107, E11, E83: value LS74 -> (none)
- E105: value LS27 -> (none)
- E108, E23, E24, E47, E77, E84: value LS08 -> (none)
- E12, E13, E15, E17, E18, E19, E20, E29, E39, E5, E6, E66, E7, E8: value LS244 -> (none)
- E14, E16: value LS367 -> (none)
- E2, E42: value LS14 -> (none)
- E21, E22, E36, E37, E80, E94: value LS04 -> (none)
- E25: value 7404 -> (none)
- E26, E27, E28: value LS38 -> (none)
- E3: value S74 -> (none)
- E30: value Z80A SIO/1 -> (none)
- E32: value Z80A CPU -> (none)
- E33: value Z80A DMA -> (none)
- E34, E38, E41, E46, E54, E91: value LS32 -> (none)
- E35: value MM58167A -> (none)
- E4, E82: value S04 -> (none)
- E40: value LS42 -> (none)
- E43, E44: value MC1488 -> (none)
- E45, E52, E53: value MC1489 -> (none)
- E48: value WD1691 -> (none)
- E49, E97: value LS157 -> (none)
- E51: value M2716 -> (none)
- E55: value LS20 -> (none)
- E56: value D765 -> (none)
- E57: value WD2143 -> (none)
- E64: value MC14411 -> (none)
- E65: value LS374 -> (none)
- E67: value Z80A CTC -> (none)
- E68, E69: value LS138 -> (none)
- E70: value LS629 -> (none)
- E78: value LS10 -> (none)
- E81: value LS01 -> (none)
- E9: value LS05 -> (none)
- E95: value LS132 -> (none)
- E96: value LS393 -> (none)
- R1, R12, R13, R22, R23, R36, R54, R55, R58, R59: value 3.3kΩ -> (none)
- R10, R37, R38, R39, R40, R41, R42: value 150Ω -> (none)
- R11: value 220Ω -> (none)
- R14, R19, R90, R94, R95: value 10kΩ -> (none)
- R15, R18, R2, R3, R4, R5, R60, R61, R62, R63, R64, R65, R66, R67, R7, R70, R71, R72, R73, R74, R75, R76, R77, R82, R85, R9: value 1kΩ -> (none)
- R16: value 56Ω -> (none)
- R17, R20: value 820Ω -> (none)
- R200: value Z 2.7V -> (none)
- R201: value 560Ω -> (none)
- R202: value 15MΩ -> (none)
- R203: value 390Ω -> (none)
- R204: value 330Ω -> (none)
- R21: value 20kΩ -> (none)
- R26: value 1.5kΩ -> (none)
- R43, R44, R45, R46, R47, R48, R49, R50, R51, R52: value 33Ω -> (none)
- R53: value 5.1kΩ -> (none)
- R68, R69, R78, R79, R80, R83, R86, R91: value 4.7kΩ -> (none)
- R84: value 47Ω -> (none)
- R87, R88: value 47kΩ -> (none)
- R89: value 68Ω -> (none)
- R92, R93: value 50kΩ -> (none)
- V1: value LED -> (none)
- V2, V3, V4: value BA513 -> (none)
- Y1: value 8MHz -> (none)
- Y2: value 32.768kHz -> (none)
- Y3: value 1.8432MHz -> (none)
Connections:
- BAT pad 1: (no net) -> GND
- BAT pad 2: (no net) -> _NET_196
- BAT pad 3: (no net) -> _NET_196
- C1 pad 1: (no net) -> 5V
- C1 pad 2: (no net) -> GND
- C10 pad 1: (no net) -> DABUS6
- C10 pad 2: (no net) -> _NET_281
- C100 pad 1: (no net) -> 5V
- C100 pad 2: (no net) -> GND
- C101 pad 1: (no net) -> _NET_288
- C101 pad 2: (no net) -> GND
- C102 pad 1: (no net) -> DISK0-
- C102 pad 2: (no net) -> GND
- C103 pad 1: (no net) -> GND
- C103 pad 2: (no net) -> BANK1-
- C11 pad 1: (no net) -> _NET_282
- C11 pad 2: (no net) -> D0
- C110 pad 1: (no net) -> 5V
- C110 pad 2: (no net) -> _NET_46
- C12 pad 1: (no net) -> _NET_283
- C12 pad 2: (no net) -> DABUS1
- C13 pad 1: (no net) -> _NET_284
- C13 pad 2: (no net) -> DABUS2
- C14 pad 1: (no net) -> _NET_285
- C14 pad 2: (no net) -> DABUS4
- C15 pad 1: (no net) -> DABUS5
- C15 pad 2: (no net) -> _NET_286
- C16 pad 1: (no net) -> DABUS3
- C16 pad 2: (no net) -> _NET_287
- C17 pad 1: (no net) -> _NET_272
- C17 pad 2: (no net) -> _NET_273
- C18 pad 1: (no net) -> _NET_268
- C18 pad 2: (no net) -> _NET_267
- C19 pad 2: (no net) -> GND
- C2 pad 1: (no net) -> 5V
- C2 pad 2: (no net) -> GND
- C20 pad 1: (no net) -> _NET_39
- C20 pad 2: (no net) -> GND
- C21 pad 1: (no net) -> GND
- C21 pad 2: (no net) -> _NET_193
- C22 pad 1: (no net) -> _NET_192
- C22 pad 2: (no net) -> GND
- C3 pad 1: (no net) -> GND
- C3 pad 2: (no net) -> -12V
- C300 pad 1: (no net) -> _NET_50
- C300 pad 2: (no net) -> _NET_49
- C301 pad 1: (no net) -> _NET_275
- C301 pad 2: (no net) -> _NET_251
- C4 pad 1: (no net) -> 12V
- C4 pad 2: (no net) -> GND
- C5 pad 1: (no net) -> _NET_36
- C5 pad 2: (no net) -> _NET_37
- C6 pad 1: (no net) -> _NET_3
- C6 pad 2: (no net) -> GND
- C7 pad 1: (no net) -> _NET_41
- C7 pad 2: (no net) -> _NET_42
- C8 pad 1: (no net) -> _NET_3
- C8 pad 2: (no net) -> GND
- C9 pad 1: (no net) -> DABUS7
- C9 pad 2: (no net) -> _NET_280
- CX1 pad 1: (no net) -> 5V
- CX1 pad 2: (no net) -> GND
- CX10 pad 1: (no net) -> 5V
- CX10 pad 2: (no net) -> GND
- CX11 pad 1: (no net) -> 5V
- CX11 pad 2: (no net) -> GND
- CX12 pad 1: (no net) -> 5V
- CX12 pad 2: (no net) -> GND
- CX13 pad 1: (no net) -> 5V
- CX13 pad 2: (no net) -> GND
- CX14 pad 1: (no net) -> GND
- CX14 pad 2: (no net) -> 5V
- CX15 pad 1: (no net) -> GND
- CX15 pad 2: (no net) -> 5V
- CX16 pad 1: (no net) -> GND
- CX16 pad 2: (no net) -> 5V
- CX17 pad 1: (no net) -> GND
- CX17 pad 2: (no net) -> 5V
- CX18 pad 1: (no net) -> 5V
- CX18 pad 2: (no net) -> GND
- CX19 pad 1: (no net) -> 5V
- CX19 pad 2: (no net) -> GND
- CX2 pad 1: (no net) -> 5V
- CX2 pad 2: (no net) -> GND
- CX20 pad 1: (no net) -> 5V
- CX20 pad 2: (no net) -> GND
- CX21 pad 1: (no net) -> 5V
- CX21 pad 2: (no net) -> GND
- CX22 pad 1: (no net) -> 5V
- CX22 pad 2: (no net) -> GND
- CX23 pad 1: (no net) -> 5V
- CX23 pad 2: (no net) -> GND
- CX24 pad 1: (no net) -> GND
- CX24 pad 2: (no net) -> 5V
- CX25 pad 1: (no net) -> GND
- CX25 pad 2: (no net) -> 5V
- CX26 pad 1: (no net) -> GND
- CX26 pad 2: (no net) -> 5V
- CX27 pad 1: (no net) -> GND
- CX27 pad 2: (no net) -> 5V
- CX28 pad 1: (no net) -> GND
- CX28 pad 2: (no net) -> 5V
- CX29 pad 1: (no net) -> 5V
- CX29 pad 2: (no net) -> GND
- CX3 pad 1: (no net) -> 5V
- CX3 pad 2: (no net) -> GND
- CX30 pad 1: (no net) -> _NET_271
- CX30 pad 2: (no net) -> GND
- CX31 pad 1: (no net) -> 5V
- CX31 pad 2: (no net) -> GND
- CX32 pad 1: (no net) -> 5V
- CX32 pad 2: (no net) -> GND
- CX33 pad 1: (no net) -> 5V
- CX33 pad 2: (no net) -> GND
- CX34 pad 1: (no net) -> 5V
- CX34 pad 2: (no net) -> GND
- CX35 pad 1: (no net) -> GND
- CX35 pad 2: (no net) -> 5V
- CX36 pad 1: (no net) -> GND
- CX36 pad 2: (no net) -> 5V
- CX37 pad 1: (no net) -> 5V
- CX37 pad 2: (no net) -> GND
- CX38 pad 1: (no net) -> 5V
- CX38 pad 2: (no net) -> GND
- CX39 pad 1: (no net) -> 5V
- CX39 pad 2: (no net) -> GND
- CX4 pad 1: (no net) -> 5V
- CX4 pad 2: (no net) -> GND
- CX40 pad 1: (no net) -> 5V
- CX40 pad 2: (no net) -> GND
- CX41 pad 1: (no net) -> 5V
- CX41 pad 2: (no net) -> unconnected-GND
- CX5 pad 1: (no net) -> 5V
- CX5 pad 2: (no net) -> GND
- CX6 pad 1: (no net) -> 5V
- CX6 pad 2: (no net) -> GND
- CX7 pad 1: (no net) -> 5V
- CX7 pad 2: (no net) -> GND
- CX8 pad 1: (no net) -> 5V
- CX8 pad 2: (no net) -> GND
- CX9 pad 1: (no net) -> 5V
- CX9 pad 2: (no net) -> GND
- E1 pad 1: (no net) -> GND
- E1 pad 10: (no net) -> unconnected-(E1-Pad10)
- E1 pad 11: (no net) -> unconnected-(E1-Pad11)
- E1 pad 12: (no net) -> unconnected-(E1-Pad12)
- E1 pad 13: (no net) -> unconnected-(E1-Pad13)
- E1 pad 14: (no net) -> _NET_36
- E1 pad 15: (no net) -> _NET_37
- E1 pad 16: (no net) -> 5V
- E1 pad 2: (no net) -> _NET_35
- E1 pad 3: (no net) -> _NET_44
- E1 pad 4: (no net) -> _NET_38
- E1 pad 5: (no net) -> unconnected-(E1-Pad5)
- E1 pad 6: (no net) -> unconnected-(E1-Pad6)
- E1 pad 7: (no net) -> unconnected-(E1-Pad7)
- E1 pad 8: (no net) -> GND
- E1 pad 9: (no net) -> unconnected-(E1-Pad9)
- E10 pad 1: (no net) -> A14I-
- E10 pad 10: (no net) -> unconnected-(E10-Pad10)
- E10 pad 11: (no net) -> _NET_47
- E10 pad 12: (no net) -> 5V
- E10 pad 13: (no net) -> unconnected-(E10-Pad13)
- E10 pad 14: (no net) -> 5V
- E10 pad 2: (no net) -> A15I-
- E10 pad 3: (no net) -> RFSHB-
- E10 pad 4: (no net) -> IORQB-
- E10 pad 5: (no net) -> 5V
- E10 pad 6: (no net) -> A13I-
- E10 pad 7: (no net) -> GND
- E10 pad 8: (no net) -> ROMSEL-
- E10 pad 9: (no net) -> unconnected-(E10-Pad9)
- E100 pad 1: (no net) -> unconnected-(E100-Pad1)
- E100 pad 10: (no net) -> _NET_77
- E100 pad 11: (no net) -> _NET_76
- E100 pad 12: (no net) -> _NET_75
- E100 pad 13: (no net) -> _NET_78
- E100 pad 14: (no net) -> D07
- E100 pad 15: (no net) -> CAS-
- E100 pad 16: (no net) -> GND
- E100 pad 2: (no net) -> DABUS7
- E100 pad 3: (no net) -> _NET_80
- E100 pad 4: (no net) -> RAS2-
- E100 pad 5: (no net) -> _NET_72
- E100 pad 6: (no net) -> _NET_74
- E100 pad 7: (no net) -> _NET_73
- E100 pad 8: (no net) -> 5V
- E100 pad 9: (no net) -> _NET_79
- E101 pad 1: (no net) -> unconnected-(E101-Pad1)
- E101 pad 10: (no net) -> _NET_77
- E101 pad 11: (no net) -> _NET_76
- E101 pad 12: (no net) -> _NET_75
- E101 pad 13: (no net) -> _NET_78
- E101 pad 14: (no net) -> D01
- E101 pad 15: (no net) -> CAS-
- E101 pad 16: (no net) -> GND
- E101 pad 2: (no net) -> DABUS1
- E101 pad 3: (no net) -> _NET_80
- E101 pad 4: (no net) -> RAS2-
- E101 pad 5: (no net) -> _NET_72
- E101 pad 6: (no net) -> _NET_74
- E101 pad 7: (no net) -> _NET_73
- E101 pad 8: (no net) -> 5V
- E101 pad 9: (no net) -> _NET_79
- E102 pad 1: (no net) -> _NET_118
- E102 pad 10: (no net) -> _NET_132
- E102 pad 11: (no net) -> _NET_146
- E102 pad 12: (no net) -> S1BA
- E102 pad 13: (no net) -> _NET_147
- E102 pad 14: (no net) -> 5V
- E102 pad 2: (no net) -> _NET_119
- E102 pad 3: (no net) -> _NET_120
- E102 pad 4: (no net) -> _NET_145
- E102 pad 5: (no net) -> _NET_143
- E102 pad 6: (no net) -> _NET_144
- E102 pad 7: (no net) -> GND
- E102 pad 8: (no net) -> _NET_127
- E102 pad 9: (no net) -> STBB
- E103 pad 1: (no net) -> RESET-
- E103 pad 10: (no net) -> 5V
- E103 pad 11: (no net) -> _NET_214
- E103 pad 12: (no net) -> _NET_218
- E103 pad 13: (no net) -> RESET-
- E103 pad 14: (no net) -> 5V
- E103 pad 2: (no net) -> _NET_216
- E103 pad 3: (no net) -> _NET_214
- E103 pad 4: (no net) -> 5V
- E103 pad 5: (no net) -> _NET_218
- E103 pad 6: (no net) -> _NET_219
- E103 pad 7: (no net) -> GND
- E103 pad 8: (no net) -> unconnected-(E103-Pad8)
- E103 pad 9: (no net) -> _NET_217
- E104 pad 1: (no net) -> 5V
- E104 pad 10: (no net) -> RESET-
- E104 pad 11: (no net) -> _NET_214
- E104 pad 12: (no net) -> 4D-
- E104 pad 13: (no net) -> 5V
- E104 pad 14: (no net) -> 5V
- E104 pad 2: (no net) -> CB-
- E104 pad 3: (no net) -> _NET_214
- E104 pad 4: (no net) -> RESET-
- E104 pad 5: (no net) -> unconnected-(E104-Pad5)
- E104 pad 6: (no net) -> _NET_213
- E104 pad 7: (no net) -> GND
- E104 pad 8: (no net) -> _NET_215
- E104 pad 9: (no net) -> unconnected-(E104-Pad9)
- E105 pad 1: (no net) -> _NET_224
- E105 pad 10: (no net) -> FDCIEI-
- E105 pad 11: (no net) -> ED-
- E105 pad 12: (no net) -> FDCIEO
- E105 pad 13: (no net) -> FDCIEI-
- E105 pad 14: (no net) -> 5V
- E105 pad 2: (no net) -> _NET_225
- E105 pad 3: (no net) -> IORQB-
- E105 pad 4: (no net) -> M1B-
- E105 pad 5: (no net) -> FDCIEI-
- E105 pad 6: (no net) -> _NET_221
- E105 pad 7: (no net) -> GND
- E105 pad 8: (no net) -> _NET_216
- E105 pad 9: (no net) -> _NET_213
- E106 pad 1: (no net) -> _NET_223
- E106 pad 10: (no net) -> 5V
- E106 pad 11: (no net) -> _NET_221
- E106 pad 12: (no net) -> _NET_226
- E106 pad 13: (no net) -> _NET_227
- E106 pad 14: (no net) -> 5V
- E106 pad 2: (no net) -> 5V
- E106 pad 3: (no net) -> FDINT+
- E106 pad 4: (no net) -> 5V
- E106 pad 5: (no net) -> _NET_226
- E106 pad 6: (no net) -> unconnected-(E106-Pad6)
- E106 pad 7: (no net) -> GND
- E106 pad 8: (no net) -> unconnected-(E106-Pad8)
- E106 pad 9: (no net) -> _NET_224
- E107 pad 1: (no net) -> 5V
- E107 pad 10: (no net) -> _NET_201
- E107 pad 11: (no net) -> 5V
- E107 pad 12: (no net) -> 5V
- E107 pad 13: (no net) -> _NET_200
- E107 pad 14: (no net) -> 5V
- E107 pad 2: (no net) -> GND
- E107 pad 3: (no net) -> WRI-
- E107 pad 4: (no net) -> _NET_198
- E107 pad 5: (no net) -> _NET_199
- E107 pad 6: (no net) -> SIG-
- E107 pad 7: (no net) -> GND
- E107 pad 8: (no net) -> unconnected-(E107-Pad8)
- E107 pad 9: (no net) -> MON
- E108 pad 1: (no net) -> _NET_258
- E108 pad 10: (no net) -> _NET_263
- E108 pad 11: (no net) -> _NET_228
- E108 pad 12: (no net) -> _NET_257
- E108 pad 13: (no net) -> BUSAKB+
- E108 pad 14: (no net) -> 5V
- E108 pad 2: (no net) -> _NET_259
- E108 pad 3: (no net) -> _NET_260
- E108 pad 4: (no net) -> _NET_260
- E108 pad 5: (no net) -> _NET_261
- E108 pad 6: (no net) -> _NET_262
- E108 pad 7: (no net) -> GND
- E108 pad 8: (no net) -> _NET_264
- E108 pad 9: (no net) -> _NET_262
- E11 pad 1: (no net) -> SEL1-
- E11 pad 10: (no net) -> _NET_53
- E11 pad 11: (no net) -> _NET_54
- E11 pad 12: (no net) -> _NET_54
- E11 pad 13: (no net) -> SEL3-
- E11 pad 14: (no net) -> 5V
- E11 pad 2: (no net) -> _NET_48
- E11 pad 3: (no net) -> _NET_48
- E11 pad 4: (no net) -> RESET-
- E11 pad 5: (no net) -> _NET_47
- E11 pad 6: (no net) -> unconnected-(E11-Pad6)
- E11 pad 7: (no net) -> GND
- E11 pad 8: (no net) -> BANKA1-
- E11 pad 9: (no net) -> BANKA2-
- E12 pad 1: (no net) -> DINB
- E12 pad 10: (no net) -> GND
- E12 pad 11: (no net) -> D6B
- E12 pad 12: (no net) -> DABUS7
- E12 pad 13: (no net) -> D4B
- E12 pad 14: (no net) -> DABUS5
- E12 pad 15: (no net) -> D2B
- E12 pad 16: (no net) -> DABUS3
- E12 pad 17: (no net) -> D0B
- E12 pad 18: (no net) -> DABUS1
- E12 pad 19: (no net) -> DINB
- E12 pad 2: (no net) -> D1B
- E12 pad 20: (no net) -> 5V
- E12 pad 3: (no net) -> D0
- E12 pad 4: (no net) -> D3B
- E12 pad 5: (no net) -> DABUS2
- E12 pad 6: (no net) -> D5B
- E12 pad 7: (no net) -> DABUS4
- E12 pad 8: (no net) -> D7B
- E12 pad 9: (no net) -> DABUS6
- E13 pad 1: (no net) -> BUSAKB-
- E13 pad 10: (no net) -> GND
- E13 pad 11: (no net) -> SEL9-
- E13 pad 12: (no net) -> MRB-
- E13 pad 13: (no net) -> MRB-
- E13 pad 14: (no net) -> RDB-
- E13 pad 15: (no net) -> RDB-
- E13 pad 16: (no net) -> IORQB-
- E13 pad 17: (no net) -> IORQB-
- E13 pad 18: (no net) -> MREQB-
- E13 pad 19: (no net) -> BUSAKB+
- E13 pad 2: (no net) -> _NET_173
- E13 pad 20: (no net) -> 5V
- E13 pad 3: (no net) -> _NET_172
- E13 pad 4: (no net) -> _NET_172
- E13 pad 5: (no net) -> _NET_171
- E13 pad 6: (no net) -> _NET_171
- E13 pad 7: (no net) -> _NET_170
- E13 pad 8: (no net) -> _NET_170
- E13 pad 9: (no net) -> _NET_169
- E14 pad 1: (no net) -> GND
- E14 pad 10: (no net) -> _NET_206
- E14 pad 11: (no net) -> unconnected-(E14-Pad11)
- E14 pad 12: (no net) -> unconnected-(E14-Pad12)
- E14 pad 13: (no net) -> D0
- E14 pad 14: (no net) -> MON
- E14 pad 15: (no net) -> _NET_210
- E14 pad 16: (no net) -> 5V
- E14 pad 2: (no net) -> BUSRQ-
- E14 pad 3: (no net) -> _NET_29
- E14 pad 4: (no net) -> WAITB-
- E14 pad 5: (no net) -> _NET_31
- E14 pad 6: (no net) -> NMI-
- E14 pad 7: (no net) -> _NET_30
- E14 pad 8: (no net) -> GND
- E14 pad 9: (no net) -> IEOB
- E15 pad 1: (no net) -> BUSAKB+
- E15 pad 10: (no net) -> GND
- E15 pad 11: (no net) -> MRB-
- E15 pad 12: (no net) -> MRB-
- E15 pad 13: (no net) -> RDB-
- E15 pad 14: (no net) -> RDB-
- E15 pad 15: (no net) -> IORQB-
- E15 pad 16: (no net) -> IORQB-
- E15 pad 17: (no net) -> 0B
- E15 pad 18: (no net) -> RFSHB-
- E15 pad 19: (no net) -> GND
- E15 pad 2: (no net) -> _NET_21
- E15 pad 20: (no net) -> 5V
- E15 pad 3: (no net) -> BI
- E15 pad 4: (no net) -> IORQ-
- E15 pad 5: (no net) -> unconnected-(E15-Pad5)
- E15 pad 6: (no net) -> _NET_23
- E15 pad 7: (no net) -> RDI-
- E15 pad 8: (no net) -> _NET_22
- E15 pad 9: (no net) -> _NET_50
- E16 pad 1: (no net) -> GND
- E16 pad 10: (no net) -> _NET_32
- E16 pad 11: (no net) -> unconnected-(E16-Pad11)
- E16 pad 12: (no net) -> unconnected-(E16-Pad12)
- E16 pad 13: (no net) -> MREQB-
- E16 pad 14: (no net) -> _NET_20
- E16 pad 15: (no net) -> BUSAKB+
- E16 pad 16: (no net) -> 5V
- E16 pad 2: (no net) -> _NET_25
- E16 pad 3: (no net) -> M1B-
- E16 pad 4: (no net) -> _NET_24
- E16 pad 5: (no net) -> BUSAKB-
- E16 pad 6: (no net) -> _NET_27
- E16 pad 7: (no net) -> HALTB-
- E16 pad 8: (no net) -> GND
- E16 pad 9: (no net) -> 0B
- E17 pad 1: (no net) -> BUSAKB+
- E17 pad 10: (no net) -> GND
- E17 pad 11: (no net) -> _NET_9
- E17 pad 12: (no net) -> A12B
- E17 pad 13: (no net) -> _NET_6
- E17 pad 14: (no net) -> A8B
- E17 pad 15: (no net) -> _NET_10
- E17 pad 16: (no net) -> A11B
- E17 pad 17: (no net) -> _NET_4
- E17 pad 18: (no net) -> A14B
- E17 pad 19: (no net) -> BUSAKB+
- E17 pad 2: (no net) -> _NET_5
- E17 pad 20: (no net) -> 5V
- E17 pad 3: (no net) -> A15B
- E17 pad 4: (no net) -> _NET_8
- E17 pad 5: (no net) -> A9B
- E17 pad 6: (no net) -> _NET_11
- E17 pad 7: (no net) -> A13B
- E17 pad 8: (no net) -> _NET_7
- E17 pad 9: (no net) -> A10B
- E18 pad 1: (no net) -> BUSAKB-
- E18 pad 10: (no net) -> GND
- E18 pad 11: (no net) -> _NET_187
- E18 pad 12: (no net) -> A12B
- E18 pad 13: (no net) -> _NET_184
- E18 pad 14: (no net) -> A8B
- E18 pad 15: (no net) -> _NET_188
- E18 pad 16: (no net) -> A11B
- E18 pad 17: (no net) -> _NET_182
- E18 pad 18: (no net) -> A14B
- E18 pad 19: (no net) -> BUSAKB-
- E18 pad 2: (no net) -> _NET_183
- E18 pad 20: (no net) -> 5V
- E18 pad 3: (no net) -> A15B
- E18 pad 4: (no net) -> _NET_186
- E18 pad 5: (no net) -> A9B
- E18 pad 6: (no net) -> _NET_189
- E18 pad 7: (no net) -> A13B
- E18 pad 8: (no net) -> _NET_185
- E18 pad 9: (no net) -> A10B
- E19 pad 1: (no net) -> GND
- E19 pad 10: (no net) -> GND
- E19 pad 11: (no net) -> A10B
- E19 pad 12: (no net) -> A12I
- E19 pad 13: (no net) -> A13B
- E19 pad 14: (no net) -> A8I
- E19 pad 15: (no net) -> A9B
- E19 pad 16: (no net) -> A11I
- E19 pad 17: (no net) -> A15B
- E19 pad 18: (no net) -> A14I
- E19 pad 19: (no net) -> GND
- E19 pad 2: (no net) -> A14B
- E19 pad 20: (no net) -> 5V
- E19 pad 3: (no net) -> A15I
- E19 pad 4: (no net) -> A11B
- E19 pad 5: (no net) -> A9I
- E19 pad 6: (no net) -> A8B
- E19 pad 7: (no net) -> A13I
- E19 pad 8: (no net) -> A12B
- E19 pad 9: (no net) -> A10I
- E2 pad 1: (no net) -> _NET_3
- E2 pad 10: (no net) -> _NET_91
- E2 pad 11: (no net) -> _NET_93
- E2 pad 12: (no net) -> _NET_93
- E2 pad 13: (no net) -> RXD1
- E2 pad 14: (no net) -> 5V
- E2 pad 2: (no net) -> _NET_2
- E2 pad 3: (no net) -> MREQB-
- E2 pad 4: (no net) -> unconnected-MREQI+
- E2 pad 5: (no net) -> unconnected-(E2-Pad5)
- E2 pad 6: (no net) -> unconnected-(E2-Pad6)
- E2 pad 7: (no net) -> GND
- E2 pad 8: (no net) -> _NET_254
- E2 pad 9: (no net) -> _NET_270
- E20 pad 1: (no net) -> MUX-
- E20 pad 10: (no net) -> GND
- E20 pad 11: (no net) -> A12I
- E20 pad 12: (no net) -> _NET_83
- E20 pad 13: (no net) -> A8I
- E20 pad 14: (no net) -> _NET_86
- E20 pad 15: (no net) -> A11I
- E20 pad 16: (no net) -> _NET_82
- E20 pad 17: (no net) -> A14I
- E20 pad 18: (no net) -> _NET_88
- E20 pad 19: (no net) -> MUX-
- E20 pad 2: (no net) -> A15I
- E20 pad 20: (no net) -> 5V
- E20 pad 3: (no net) -> _NET_87
- E20 pad 4: (no net) -> A9I
- E20 pad 5: (no net) -> _NET_84
- E20 pad 6: (no net) -> A13I
- E20 pad 7: (no net) -> _NET_81
- E20 pad 8: (no net) -> A10I
- E20 pad 9: (no net) -> _NET_85
- E21 pad 1: (no net) -> _NET_208
- E21 pad 10: (no net) -> A15I-
- E21 pad 11: (no net) -> A15I
- E21 pad 12: (no net) -> unconnected-(E21-Pad12)
- E21 pad 13: (no net) -> unconnected-(E21-Pad13)
- E21 pad 14: (no net) -> 5V
- E21 pad 2: (no net) -> _NET_190
- E21 pad 3: (no net) -> A14I
- E21 pad 4: (no net) -> A14I-
- E21 pad 5: (no net) -> _NET_191
- E21 pad 6: (no net) -> _NET_207
- E21 pad 7: (no net) -> GND
- E21 pad 8: (no net) -> A13I-
- E21 pad 9: (no net) -> A13I
- E22 pad 1: (no net) -> _NET_50
- E22 pad 10: (no net) -> _NET_277
- E22 pad 11: (no net) -> DS1
- E22 pad 12: (no net) -> _NET_45
- E22 pad 13: (no net) -> IORQ-
- E22 pad 14: (no net) -> 5V
- E22 pad 2: (no net) -> _NET_49
- E22 pad 3: (no net) -> _NET_49
- E22 pad 4: (no net) -> WRI-
- E22 pad 5: (no net) -> BUSAKB-
- E22 pad 6: (no net) -> BUSAKB+
- E22 pad 7: (no net) -> GND
- E22 pad 8: (no net) -> _NET_288
- E22 pad 9: (no net) -> _NET_279
- E23 pad 1: (no net) -> _NET_59
- E23 pad 10: (no net) -> _NET_65
- E23 pad 11: (no net) -> _NET_71
- E23 pad 12: (no net) -> _NET_70
- E23 pad 13: (no net) -> _NET_70
- E23 pad 14: (no net) -> 5V
- E23 pad 2: (no net) -> _NET_58
- E23 pad 3: (no net) -> RAS2-
- E23 pad 4: (no net) -> unconnected-(E23-Pad4)
- E23 pad 5: (no net) -> unconnected-(E23-Pad5)
- E23 pad 6: (no net) -> unconnected-(E23-Pad6)
- E23 pad 7: (no net) -> GND
- E23 pad 8: (no net) -> RAS1-
- E23 pad 9: (no net) -> _NET_58
- E24 pad 1: (no net) -> _NET_55
- E24 pad 10: (no net) -> RESET-
- E24 pad 11: (no net) -> _NET_46
- E24 pad 12: (no net) -> _NET_45
- E24 pad 13: (no net) -> M1B-
- E24 pad 14: (no net) -> 5V
- E24 pad 2: (no net) -> BANKA1-
- E24 pad 3: (no net) -> BANK1-
- E24 pad 4: (no net) -> A15I
- E24 pad 5: (no net) -> A14I
- E24 pad 6: (no net) -> _NET_56
- E24 pad 7: (no net) -> GND
- E24 pad 8: (no net) -> _NET_53
- E24 pad 9: (no net) -> SEL2-
- E25 pad 1: (no net) -> _NET_67
- E25 pad 10: (no net) -> _NET_66
- E25 pad 11: (no net) -> MUX+
- E25 pad 12: (no net) -> MUX+
- E25 pad 13: (no net) -> SIGN1-
- E25 pad 14: (no net) -> 5V
- E25 pad 2: (no net) -> _NET_68
- E25 pad 3: (no net) -> _NET_68
- E25 pad 4: (no net) -> _NET_69
- E25 pad 5: (no net) -> _NET_66
- E25 pad 6: (no net) -> _NET_67
- E25 pad 7: (no net) -> GND
- E25 pad 8: (no net) -> _NET_70
- E25 pad 9: (no net) -> _NET_69
- E26 pad 1: (no net) -> DS1
- E26 pad 10: (no net) -> _NET_237
- E26 pad 11: (no net) -> HEADSEL-
- E26 pad 12: (no net) -> HDSEL
- E26 pad 13: (no net) -> HDSEL
- E26 pad 14: (no net) -> 5V
- E26 pad 2: (no net) -> _NET_276
- E26 pad 3: (no net) -> DISK2-
- E26 pad 4: (no net) -> DS0
- E26 pad 5: (no net) -> _NET_277
- E26 pad 6: (no net) -> DISK1-
- E26 pad 7: (no net) -> GND
- E26 pad 8: (no net) -> WRITEEN-
- E26 pad 9: (no net) -> _NET_237
- E27 pad 1: (no net) -> LC-DIR
- E27 pad 10: (no net) -> _NET_248
- E27 pad 11: (no net) -> STEP-
- E27 pad 12: (no net) -> FR-STP
- E27 pad 13: (no net) -> SEEK
- E27 pad 14: (no net) -> 5V
- E27 pad 2: (no net) -> SEEK
- E27 pad 3: (no net) -> DIRECTION-
- E27 pad 4: (no net) -> MON
- E27 pad 5: (no net) -> MON
- E27 pad 6: (no net) -> MOTORON-
- E27 pad 7: (no net) -> GND
- E27 pad 8: (no net) -> WDATA-
- E27 pad 9: (no net) -> _NET_248
- E28 pad 1: (no net) -> DS1
- E28 pad 10: (no net) -> HDL
- E28 pad 11: (no net) -> unconnected-(E28-Pad11)
- E28 pad 12: (no net) -> FR-STP
- E28 pad 13: (no net) -> SEEK-
- E28 pad 14: (no net) -> 5V
- E28 pad 2: (no net) -> DS0
- E28 pad 3: (no net) -> DISK4-
- E28 pad 4: (no net) -> _NET_276
- E28 pad 5: (no net) -> _NET_277
- E28 pad 6: (no net) -> DISK0-
- E28 pad 7: (no net) -> GND
- E28 pad 8: (no net) -> unconnected-HEADLOAD-
- E28 pad 9: (no net) -> HDL
- E29 pad 1: (no net) -> WRI-
- E29 pad 10: (no net) -> GND
- E29 pad 11: (no net) -> DABUS1
- E29 pad 12: (no net) -> D0B
- E29 pad 13: (no net) -> DABUS3
- E29 pad 14: (no net) -> D2B
- E29 pad 15: (no net) -> DABUS5
- E29 pad 16: (no net) -> D4B
- E29 pad 17: (no net) -> DABUS7
- E29 pad 18: (no net) -> D6B
- E29 pad 19: (no net) -> WRI-
- E29 pad 2: (no net) -> DABUS6
- E29 pad 20: (no net) -> 5V
- E29 pad 3: (no net) -> D7B
- E29 pad 4: (no net) -> DABUS4
- E29 pad 5: (no net) -> D5B
- E29 pad 6: (no net) -> DABUS2
- E29 pad 7: (no net) -> D3B
- E29 pad 8: (no net) -> D0
- E29 pad 9: (no net) -> D1B
- E3 pad 1: (no net) -> _NET_33
- E3 pad 10: (no net) -> _NET_44
- E3 pad 11: (no net) -> _NET_1
- E3 pad 12: (no net) -> _NET_44
- E3 pad 13: (no net) -> _NET_2
- E3 pad 14: (no net) -> 5V
- E3 pad 2: (no net) -> _NET_32
- E3 pad 3: (no net) -> _NET_34
- E3 pad 4: (no net) -> _NET_33
- E3 pad 5: (no net) -> unconnected-(E3-Pad5)
- E3 pad 6: (no net) -> _NET_32
- E3 pad 7: (no net) -> GND
- E3 pad 8: (no net) -> unconnected-(E3-Pad8)
- E3 pad 9: (no net) -> _NET_35
- E30 pad 1: (no net) -> DABUS1
- E30 pad 10: (no net) -> unconnected-(E30-Pad10)
- E30 pad 11: (no net) -> unconnected-(E30-Pad11)
- E30 pad 12: (no net) -> _NET_91
- E30 pad 13: (no net) -> SPEED1
- E30 pad 14: (no net) -> SPEED1
- E30 pad 15: (no net) -> _NET_92
- E30 pad 16: (no net) -> unconnected-(E30-Pad16)
- E30 pad 17: (no net) -> unconnected-(E30-Pad17)
- E30 pad 18: (no net) -> unconnected-(E30-Pad18)
- E30 pad 19: (no net) -> unconnected-(E30-Pad19)
- E30 pad 2: (no net) -> DABUS3
- E30 pad 20: (no net) -> BI
- E30 pad 21: (no net) -> RESET-
- E30 pad 22: (no net) -> _NET_98
- E30 pad 23: (no net) -> _NET_97
- E30 pad 24: (no net) -> _NET_96
- E30 pad 25: (no net) -> _NET_95
- E30 pad 26: (no net) -> SPEED2
- E30 pad 27: (no net) -> SPEED2
- E30 pad 28: (no net) -> _NET_94
- E30 pad 29: (no net) -> unconnected-(E30-Pad29)
- E30 pad 3: (no net) -> DABUS5
- E30 pad 30: (no net) -> unconnected-(E30-Pad30)
- E30 pad 31: (no net) -> GND
- E30 pad 32: (no net) -> RDI-
- E30 pad 33: (no net) -> A0I
- E30 pad 34: (no net) -> A1I
- E30 pad 35: (no net) -> SEL12-
- E30 pad 36: (no net) -> IORQB-
- E30 pad 37: (no net) -> DABUS6
- E30 pad 38: (no net) -> DABUS4
- E30 pad 39: (no net) -> DABUS2
- E30 pad 4: (no net) -> DABUS7
- E30 pad 40: (no net) -> D0
- E30 pad 5: (no net) -> INT-
- E30 pad 6: (no net) -> SIOIEI1
- E30 pad 7: (no net) -> SIOIEO1
- E30 pad 8: (no net) -> M1B-
- E30 pad 9: (no net) -> 5V
- E31 pad 1: (no net) -> DABUS1
- E31 pad 10: (no net) -> unconnected-(E31-Pad10)
- E31 pad 11: (no net) -> unconnected-(E31-Pad11)
- E31 pad 12: (no net) -> _NET_102
- E31 pad 13: (no net) -> SPEED3
- E31 pad 14: (no net) -> SPEED3
- E31 pad 15: (no net) -> _NET_103
- E31 pad 16: (no net) -> unconnected-(E31-Pad16)
- E31 pad 17: (no net) -> _NET_104
- E31 pad 18: (no net) -> _NET_105
- E31 pad 19: (no net) -> _NET_106
- E31 pad 2: (no net) -> DABUS3
- E31 pad 20: (no net) -> BI
- E31 pad 21: (no net) -> RESET-
- E31 pad 22: (no net) -> _NET_111
- E31 pad 23: (no net) -> _NET_110
- E31 pad 24: (no net) -> _NET_109
- E31 pad 25: (no net) -> _NET_108
- E31 pad 26: (no net) -> SPEED4
- E31 pad 27: (no net) -> SPEED4
- E31 pad 28: (no net) -> _NET_107
- E31 pad 29: (no net) -> unconnected-(E31-Pad29)
- E31 pad 3: (no net) -> DABUS5
- E31 pad 30: (no net) -> unconnected-(E31-Pad30)
- E31 pad 31: (no net) -> GND
- E31 pad 32: (no net) -> RDI-
- E31 pad 33: (no net) -> A0I
- E31 pad 34: (no net) -> A1I
- E31 pad 35: (no net) -> SEL13-
- E31 pad 36: (no net) -> IORQB-
- E31 pad 37: (no net) -> DABUS6
- E31 pad 38: (no net) -> DABUS4
- E31 pad 39: (no net) -> DABUS2
- E31 pad 4: (no net) -> DABUS7
- E31 pad 40: (no net) -> D0
- E31 pad 5: (no net) -> INT-
- E31 pad 6: (no net) -> SIOIEI2
- E31 pad 7: (no net) -> SIOIEO2
- E31 pad 8: (no net) -> M1B-
- E31 pad 9: (no net) -> 5V
- E32 pad 1: (no net) -> _NET_8
- E32 pad 10: (no net) -> DABUS6
- E32 pad 11: (no net) -> 5V
- E32 pad 12: (no net) -> DABUS2
- E32 pad 13: (no net) -> DABUS7
- E32 pad 14: (no net) -> D0
- E32 pad 15: (no net) -> DABUS1
- E32 pad 16: (no net) -> _NET_28
- E32 pad 17: (no net) -> _NET_30
- E32 pad 18: (no net) -> _NET_27
- E32 pad 19: (no net) -> _NET_20
- E32 pad 2: (no net) -> _NET_7
- E32 pad 20: (no net) -> IORQ-
- E32 pad 21: (no net) -> _NET_23
- E32 pad 22: (no net) -> _NET_22
- E32 pad 23: (no net) -> _NET_24
- E32 pad 24: (no net) -> _NET_31
- E32 pad 25: (no net) -> _NET_29
- E32 pad 26: (no net) -> RESET-
- E32 pad 27: (no net) -> _NET_25
- E32 pad 28: (no net) -> _NET_21
- E32 pad 29: (no net) -> GND
- E32 pad 3: (no net) -> _NET_6
- E32 pad 30: (no net) -> _NET_19
- E32 pad 31: (no net) -> _NET_18
- E32 pad 32: (no net) -> _NET_17
- E32 pad 33: (no net) -> _NET_16
- E32 pad 34: (no net) -> _NET_15
- E32 pad 35: (no net) -> _NET_14
- E32 pad 36: (no net) -> _NET_13
- E32 pad 37: (no net) -> _NET_12
- E32 pad 38: (no net) -> _NET_11
- E32 pad 39: (no net) -> _NET_10
- E32 pad 4: (no net) -> _NET_5
- E32 pad 40: (no net) -> _NET_9
- E32 pad 5: (no net) -> _NET_4
- E32 pad 6: (no net) -> _NET_32
- E32 pad 7: (no net) -> DABUS4
- E32 pad 8: (no net) -> DABUS3
- E32 pad 9: (no net) -> DABUS5
- E33 pad 1: (no net) -> _NET_176
- E33 pad 10: (no net) -> _NET_172
- E33 pad 11: (no net) -> 5V
- E33 pad 12: (no net) -> _NET_173
- E33 pad 13: (no net) -> unconnected-(E33-Pad13)
- E33 pad 14: (no net) -> BUSAKB-
- E33 pad 15: (no net) -> BUSRQ-
- E33 pad 16: (no net) -> _NET_169
- E33 pad 17: (no net) -> _NET_182
- E33 pad 18: (no net) -> _NET_183
- E33 pad 19: (no net) -> _NET_184
- E33 pad 2: (no net) -> _NET_177
- E33 pad 20: (no net) -> _NET_185
- E33 pad 21: (no net) -> _NET_186
- E33 pad 22: (no net) -> _NET_187
- E33 pad 23: (no net) -> _NET_188
- E33 pad 24: (no net) -> _NET_189
- E33 pad 25: (no net) -> _NET_168
- E33 pad 26: (no net) -> M1B-
- E33 pad 27: (no net) -> DABUS7
- E33 pad 28: (no net) -> DABUS6
- E33 pad 29: (no net) -> DABUS5
- E33 pad 3: (no net) -> _NET_178
- E33 pad 30: (no net) -> GND
- E33 pad 31: (no net) -> DABUS4
- E33 pad 32: (no net) -> DABUS3
- E33 pad 33: (no net) -> DABUS2
- E33 pad 34: (no net) -> DABUS1
- E33 pad 35: (no net) -> D0
- E33 pad 36: (no net) -> DMAIEO
- E33 pad 37: (no net) -> INT1-
- E33 pad 38: (no net) -> CTCIEO
- E33 pad 39: (no net) -> _NET_174
- E33 pad 4: (no net) -> _NET_179
- E33 pad 40: (no net) -> _NET_175
- E33 pad 5: (no net) -> _NET_180
- E33 pad 6: (no net) -> _NET_181
- E33 pad 7: (no net) -> BI
- E33 pad 8: (no net) -> _NET_170
- E33 pad 9: (no net) -> _NET_171
- E34 pad 1: (no net) -> _NET_205
- E34 pad 10: (no net) -> unconnected-(E34-Pad10)
- E34 pad 11: (no net) -> DACK-
- E34 pad 12: (no net) -> SIG-
- E34 pad 13: (no net) -> BUSAKB-
- E34 pad 14: (no net) -> 5V
- E34 pad 2: (no net) -> _NET_199
- E34 pad 3: (no net) -> _NET_168
- E34 pad 4: (no net) -> unconnected-(E34-Pad4)
- E34 pad 5: (no net) -> unconnected-(E34-Pad5)
- E34 pad 6: (no net) -> unconnected-(E34-Pad6)
- E34 pad 7: (no net) -> GND
- E34 pad 8: (no net) -> unconnected-(E34-Pad8)
- E34 pad 9: (no net) -> unconnected-(E34-Pad9)
- E35 pad 1: (no net) -> _NET_190
- E35 pad 10: (no net) -> _NET_192
- E35 pad 11: (no net) -> _NET_193
- E35 pad 12: (no net) -> GND
- E35 pad 13: (no net) -> _NET_194
- E35 pad 14: (no net) -> unconnected-(E35-Pad14)
- E35 pad 15: (no net) -> D0
- E35 pad 16: (no net) -> DABUS1
- E35 pad 17: (no net) -> DABUS2
- E35 pad 18: (no net) -> DABUS3
- E35 pad 19: (no net) -> DABUS4
- E35 pad 2: (no net) -> RDI-
- E35 pad 20: (no net) -> DABUS5
- E35 pad 21: (no net) -> DABUS6
- E35 pad 22: (no net) -> DABUS7
- E35 pad 23: (no net) -> RESET
- E35 pad 24: (no net) -> _NET_195
- E35 pad 3: (no net) -> WRI-
- E35 pad 4: (no net) -> _NET_191
- E35 pad 5: (no net) -> A0I
- E35 pad 6: (no net) -> A1I
- E35 pad 7: (no net) -> A2I
- E35 pad 8: (no net) -> A3I
- E35 pad 9: (no net) -> A4I
- E36 pad 1: (no net) -> ROMSEL-
- E36 pad 10: (no net) -> _NET_61
- E36 pad 11: (no net) -> RFSHB-
- E36 pad 12: (no net) -> _NET_64
- E36 pad 13: (no net) -> MREQB-
- E36 pad 14: (no net) -> 5V
- E36 pad 2: (no net) -> _NET_62
- E36 pad 3: (no net) -> _NET_64
- E36 pad 4: (no net) -> _NET_63
- E36 pad 5: (no net) -> MUX+
- E36 pad 6: (no net) -> MUX-
- E36 pad 7: (no net) -> GND
- E36 pad 8: (no net) -> _NET_55
- E36 pad 9: (no net) -> _NET_56
- E37 pad 1: (no net) -> _NET_235
- E37 pad 10: (no net) -> _NET_51
- E37 pad 11: (no net) -> _NET_46
- E37 pad 12: (no net) -> _NET_257
- E37 pad 13: (no net) -> INT1-
- E37 pad 14: (no net) -> 5V
- E37 pad 2: (no net) -> MFM-
- E37 pad 3: (no net) -> A6I
- E37 pad 4: (no net) -> _NET_52
- E37 pad 5: (no net) -> DMARQ-
- E37 pad 6: (no net) -> _NET_205
- E37 pad 7: (no net) -> GND
- E37 pad 8: (no net) -> _NET_242
- E37 pad 9: (no net) -> _NET_240
- E38 pad 1: (no net) -> BANK2-
- E38 pad 10: (no net) -> _NET_61
- E38 pad 11: (no net) -> _NET_90
- E38 pad 12: (no net) -> SIGN1-
- E38 pad 13: (no net) -> RDI-
- E38 pad 14: (no net) -> 5V
- E38 pad 2: (no net) -> _NET_57
- E38 pad 3: (no net) -> _NET_59
- E38 pad 4: (no net) -> BANK1-
- E38 pad 5: (no net) -> _NET_57
- E38 pad 6: (no net) -> _NET_65
- E38 pad 7: (no net) -> GND
- E38 pad 8: (no net) -> SIGN1-
- E38 pad 9: (no net) -> _NET_60
- E39 pad 1: (no net) -> _NET_89
- E39 pad 10: (no net) -> GND
- E39 pad 11: (no net) -> D06
- E39 pad 12: (no net) -> DABUS7
- E39 pad 13: (no net) -> D05
- E39 pad 14: (no net) -> D0
- E39 pad 15: (no net) -> D04
- E39 pad 16: (no net) -> DABUS1
- E39 pad 17: (no net) -> D03
- E39 pad 18: (no net) -> DABUS2
- E39 pad 19: (no net) -> _NET_89
- E39 pad 2: (no net) -> D02
- E39 pad 20: (no net) -> 5V
- E39 pad 3: (no net) -> DABUS3
- E39 pad 4: (no net) -> D01
- E39 pad 5: (no net) -> DABUS4
- E39 pad 6: (no net) -> D00
- E39 pad 7: (no net) -> DABUS5
- E39 pad 8: (no net) -> D07
- E39 pad 9: (no net) -> DABUS6
- E4 pad 1: (no net) -> CLCK
- E4 pad 10: (no net) -> _NET_42
- E4 pad 11: (no net) -> _NET_43
- E4 pad 12: (no net) -> _NET_40
- E4 pad 13: (no net) -> _NET_41
- E4 pad 14: (no net) -> 5V
- E4 pad 2: (no net) -> _NET_34
- E4 pad 3: (no net) -> M1B-
- E4 pad 4: (no net) -> _NET_1
- E4 pad 5: (no net) -> RESET+
- E4 pad 6: (no net) -> RESET-
- E4 pad 7: (no net) -> GND
- E4 pad 8: (no net) -> CLCK
- E4 pad 9: (no net) -> _NET_40
- E40 pad 1: (no net) -> ROM1-
- E40 pad 10: (no net) -> unconnected-(E40-Pad10)
- E40 pad 11: (no net) -> unconnected-(E40-Pad11)
- E40 pad 12: (no net) -> ROMSEL-
- E40 pad 13: (no net) -> RDI-
- E40 pad 14: (no net) -> A12I
- E40 pad 15: (no net) -> A11I
- E40 pad 16: (no net) -> 5V
- E40 pad 2: (no net) -> ROM2-
- E40 pad 3: (no net) -> unconnected-(E40-Pad3)
- E40 pad 4: (no net) -> unconnected-(E40-Pad4)
- E40 pad 5: (no net) -> unconnected-(E40-Pad5)
- E40 pad 6: (no net) -> unconnected-(E40-Pad6)
- E40 pad 7: (no net) -> unconnected-(E40-Pad7)
- E40 pad 8: (no net) -> GND
- E40 pad 9: (no net) -> unconnected-(E40-Pad9)
- E41 pad 1: (no net) -> _NET_63
- E41 pad 10: (no net) -> _NET_56
- E41 pad 11: (no net) -> unconnected-(E41-Pad11)
- E41 pad 12: (no net) -> unconnected-(E41-Pad12)
- E41 pad 13: (no net) -> unconnected-(E41-Pad13)
- E41 pad 14: (no net) -> 5V
- E41 pad 2: (no net) -> _NET_62
- E41 pad 3: (no net) -> _NET_57
- E41 pad 4: (no net) -> MREQB-
- E41 pad 5: (no net) -> RFSHB-
- E41 pad 6: (no net) -> _NET_58
- E41 pad 7: (no net) -> GND
- E41 pad 8: (no net) -> BANK2-
- E41 pad 9: (no net) -> BANKA2-
- E42 pad 1: (no net) -> KAWDATA-
- E42 pad 10: (no net) -> _NET_255
- E42 pad 11: (no net) -> TR00-
- E42 pad 12: (no net) -> _NET_253
- E42 pad 13: (no net) -> WRPROT-
- E42 pad 14: (no net) -> 5V
- E42 pad 2: (no net) -> _NET_256
- E42 pad 3: (no net) -> INDEX-
- E42 pad 4: (no net) -> _NET_233
- E42 pad 5: (no net) -> TWOSIDE-
- E42 pad 6: (no net) -> _NET_252
- E42 pad 7: (no net) -> GND
- E42 pad 8: (no net) -> _NET_232
- E42 pad 9: (no net) -> READY-
- E43 pad 1: (no net) -> -12V
- E43 pad 10: (no net) -> 5V
- E43 pad 11: (no net) -> RTS4
- E43 pad 12: (no net) -> _NET_109
- E43 pad 13: (no net) -> 5V
- E43 pad 14: (no net) -> 12V
- E43 pad 2: (no net) -> _NET_95
- E43 pad 3: (no net) -> TXD2
- E43 pad 4: (no net) -> _NET_96
- E43 pad 5: (no net) -> 5V
- E43 pad 6: (no net) -> RTS2
- E43 pad 7: (no net) -> GND
- E43 pad 8: (no net) -> TXD4
- E43 pad 9: (no net) -> _NET_108
- E44 pad 1: (no net) -> -12V
- E44 pad 10: (no net) -> 5V
- E44 pad 11: (no net) -> RTS3
- E44 pad 12: (no net) -> _NET_104
- E44 pad 13: (no net) -> 5V
- E44 pad 14: (no net) -> 12V
- E44 pad 2: (no net) -> unconnected-(E44-Pad2)
- E44 pad 3: (no net) -> unconnected-(E44-Pad3)
- E44 pad 4: (no net) -> unconnected-(E44-Pad4)
- E44 pad 5: (no net) -> unconnected-(E44-Pad5)
- E44 pad 6: (no net) -> unconnected-(E44-Pad6)
- E44 pad 7: (no net) -> GND
- E44 pad 8: (no net) -> TXD3
- E44 pad 9: (no net) -> _NET_103
- E45 pad 1: (no net) -> RXD2
- E45 pad 10: (no net) -> DSR2
- E45 pad 11: (no net) -> _NET_101
- E45 pad 12: (no net) -> unconnected-(E45-Pad12)
- E45 pad 13: (no net) -> DCD2
- E45 pad 14: (no net) -> 5V
- E45 pad 2: (no net) -> unconnected-(E45-Pad2)
- E45 pad 3: (no net) -> _NET_94
- E45 pad 4: (no net) -> CTS2
- E45 pad 5: (no net) -> unconnected-(E45-Pad5)
- E45 pad 6: (no net) -> _NET_99
- E45 pad 7: (no net) -> GND
- E45 pad 8: (no net) -> _NET_100
- E45 pad 9: (no net) -> unconnected-(E45-Pad9)
- E46 pad 1: (no net) -> unconnected-(E46-Pad1)
- E46 pad 10: (no net) -> _NET_99
- E46 pad 11: (no net) -> _NET_98
- E46 pad 12: (no net) -> _NET_101
- E46 pad 13: (no net) -> _NET_100
- E46 pad 14: (no net) -> 5V
- E46 pad 2: (no net) -> unconnected-(E46-Pad2)
- E46 pad 3: (no net) -> unconnected-(E46-Pad3)
- E46 pad 4: (no net) -> _NET_92
- E46 pad 5: (no net) -> _NET_92
- E46 pad 6: (no net) -> TXD1
- E46 pad 7: (no net) -> GND
- E46 pad 8: (no net) -> _NET_97
- E46 pad 9: (no net) -> _NET_100
- E47 pad 1: (no net) -> CTCIEO
- E47 pad 10: (no net) -> CTCIEO
- E47 pad 11: (no net) -> PIOIEI
- E47 pad 12: (no net) -> SIOIEO2
- E47 pad 13: (no net) -> CTCIEO
- E47 pad 14: (no net) -> 5V
- E47 pad 2: (no net) -> DMAIEO
- E47 pad 3: (no net) -> SIOIEI1
- E47 pad 4: (no net) -> CTCIEO
- E47 pad 5: (no net) -> SIOIEO1
- E47 pad 6: (no net) -> SIOIEI2
- E47 pad 7: (no net) -> GND
- E47 pad 8: (no net) -> _NET_197
- E47 pad 9: (no net) -> PIOIEO
- E48 pad 1: (no net) -> _NET_241
- E48 pad 10: (no net) -> GND
- E48 pad 11: (no net) -> _NET_249
- E48 pad 12: (no net) -> _NET_236
- E48 pad 13: (no net) -> _NET_251
- E48 pad 14: (no net) -> _NET_251
- E48 pad 15: (no net) -> MFM-
- E48 pad 16: (no net) -> _NET_250
- E48 pad 17: (no net) -> _NET_238
- E48 pad 18: (no net) -> _NET_239
- E48 pad 19: (no net) -> _NET_244
- E48 pad 2: (no net) -> _NET_246
- E48 pad 20: (no net) -> 5V
- E48 pad 3: (no net) -> _NET_245
- E48 pad 4: (no net) -> _NET_247
- E48 pad 5: (no net) -> _NET_243
- E48 pad 6: (no net) -> _NET_248
- E48 pad 7: (no net) -> _NET_237
- E48 pad 8: (no net) -> _NET_242
- E48 pad 9: (no net) -> unconnected-(E48-Pad9)
- E49 pad 1: (no net) -> SEEK
- E49 pad 10: (no net) -> unconnected-(E49-Pad10)
- E49 pad 11: (no net) -> unconnected-(E49-Pad11)
- E49 pad 12: (no net) -> unconnected-(E49-Pad12)
- E49 pad 13: (no net) -> unconnected-(E49-Pad13)
- E49 pad 14: (no net) -> unconnected-(E49-Pad14)
- E49 pad 15: (no net) -> GND
- E49 pad 16: (no net) -> 5V
- E49 pad 2: (no net) -> _NET_253
- E49 pad 3: (no net) -> _NET_252
- E49 pad 4: (no net) -> _NET_231
- E49 pad 5: (no net) -> _NET_254
- E49 pad 6: (no net) -> _NET_255
- E49 pad 7: (no net) -> _NET_230
- E49 pad 8: (no net) -> GND
- E49 pad 9: (no net) -> unconnected-(E49-Pad9)
- E5 pad 1: (no net) -> BUSAKB+
- E5 pad 10: (no net) -> GND
- E5 pad 11: (no net) -> _NET_17
- E5 pad 12: (no net) -> A4B
- E5 pad 13: (no net) -> _NET_14
- E5 pad 14: (no net) -> A0B
- E5 pad 15: (no net) -> _NET_18
- E5 pad 16: (no net) -> A3B
- E5 pad 17: (no net) -> _NET_12
- E5 pad 18: (no net) -> A6B
- E5 pad 19: (no net) -> BUSAKB+
- E5 pad 2: (no net) -> _NET_13
- E5 pad 20: (no net) -> 5V
- E5 pad 3: (no net) -> A7B
- E5 pad 4: (no net) -> _NET_16
- E5 pad 5: (no net) -> A1B
- E5 pad 6: (no net) -> _NET_19
- E5 pad 7: (no net) -> A5B
- E5 pad 8: (no net) -> _NET_15
- E5 pad 9: (no net) -> A2B
- E50 pad 1: (no net) -> A7I
- E50 pad 10: (no net) -> DABUS1
- E50 pad 11: (no net) -> DABUS2
- E50 pad 12: (no net) -> GND
- E50 pad 13: (no net) -> DABUS3
- E50 pad 14: (no net) -> DABUS4
- E50 pad 15: (no net) -> DABUS5
- E50 pad 16: (no net) -> DABUS6
- E50 pad 17: (no net) -> DABUS7
- E50 pad 18: (no net) -> ROM2-
- E50 pad 19: (no net) -> A10I
- E50 pad 2: (no net) -> A6I
- E50 pad 20: (no net) -> ROM2-
- E50 pad 21: (no net) -> 5V
- E50 pad 22: (no net) -> A9I
- E50 pad 23: (no net) -> A8I
- E50 pad 24: (no net) -> 5V
- E50 pad 3: (no net) -> A5I
- E50 pad 4: (no net) -> A4I
- E50 pad 5: (no net) -> A3I
- E50 pad 6: (no net) -> A2I
- E50 pad 7: (no net) -> A1I
- E50 pad 8: (no net) -> A0I
- E50 pad 9: (no net) -> D0
- E51 pad 1: (no net) -> A7I
- E51 pad 10: (no net) -> DABUS1
- E51 pad 11: (no net) -> DABUS2
- E51 pad 12: (no net) -> GND
- E51 pad 13: (no net) -> DABUS3
- E51 pad 14: (no net) -> DABUS4
- E51 pad 15: (no net) -> DABUS5
- E51 pad 16: (no net) -> DABUS6
- E51 pad 17: (no net) -> DABUS7
- E51 pad 18: (no net) -> ROM1-
- E51 pad 19: (no net) -> A10I
- E51 pad 2: (no net) -> A6I
- E51 pad 20: (no net) -> ROM1-
- E51 pad 21: (no net) -> 5V
- E51 pad 22: (no net) -> A9I
- E51 pad 23: (no net) -> A8I
- E51 pad 24: (no net) -> 5V
- E51 pad 3: (no net) -> A5I
- E51 pad 4: (no net) -> A4I
- E51 pad 5: (no net) -> A3I
- E51 pad 6: (no net) -> A2I
- E51 pad 7: (no net) -> A1I
- E51 pad 8: (no net) -> A0I
- E51 pad 9: (no net) -> D0
- E52 pad 1: (no net) -> RXD3
- E52 pad 10: (no net) -> DSR3
- E52 pad 11: (no net) -> _NET_114
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Routing:
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